Commit message: Updated Core URDF

File: description/robot_core.xacro (robot description, xacro)
@@ -1,5 +1,15 @@
 <?xml version="1.0"?>
 <robot xmlns:xacro="http://www.ros.org/wiki/xacro">
+    <!-- Include Inertial Macros -->
     <xacro:include filename="inertial_macros.xacro"/>
+    <!-- Define Reusable Properties -->
+    <xacro:property name="chassis_size" value="0.3 0.3 0.15"/>
+    <xacro:property name="chassis_mass" value="0.5"/>
+    <xacro:property name="wheel_radius" value="0.06"/>
+    <xacro:property name="wheel_length" value="0.04"/>
+    <xacro:property name="wheel_mass" value="0.1"/>
+    <xacro:property name="caster_radius" value="0.05"/>
+    <xacro:property name="caster_mass" value="0.1"/>
+    <!-- Define Materials -->
     <material name="white">
         <color rgba="1 1 1 1"/>
@@ -14,6 +24,8 @@
         <color rgba="0 0 0 1"/>
     </material>
+    <!-- Base Link -->
     <link name="base_link">
     </link>
+    <!-- Chassis -->
     <joint name="chassis_joint" type="fixed">
         <parent link="base_link"/>
@@ -21,22 +33,31 @@
         <origin xyz="-0.1 0 0"/>
     </joint>
+    <xacro:property name="chassis_length" value="0.4"/>
+    <xacro:property name="chassis_width" value="0.3"/>
+    <xacro:property name="chassis_height" value="0.15"/>
+    <xacro:property name="chassis_mass" value="2.0"/>
     <link name="chassis">
         <visual>
             <origin xyz="0.15 0 0.075"/>
             <geometry>
-                <box size="0.3 0.3 0.15"/>
+                <box size="${chassis_length} ${chassis_width} ${chassis_height}"/>
             </geometry>
-            <material name="white"/>
+            <material name="Metal">
+                <color rgba="0.7 0.7 0.7 1.0"/>
+            </material>
         </visual>
         <collision>
             <origin xyz="0.15 0 0.075"/>
             <geometry>
-                <box size="0.3 0.3 0.15"/>
+                <box size="${chassis_length} ${chassis_width} ${chassis_height}"/>
             </geometry>
         </collision>
-        <xacro:inertial_box mass="0.5" x="0.3" y="0.3" z=".15">
-            <origin xyz="0.15 0 0.075" rpy="0 0 0"/>
-        </xacro:inertial_box>
+        <inertial>
+            <origin xyz="0.15 0 0.075"/>
+            <mass value="${chassis_mass}"/>
+            <inertia ixx="0.1" ixy="0.0" ixz="0.0" iyy="0.1" iyz="0.0" izz="0.1"/>
+        </inertial>
     </link>
+    <!-- Left Wheel -->
     <joint name="left_wheel_joint" type="continuous">
         <parent link="base_link"/>
@@ -48,5 +69,5 @@
         <visual>
             <geometry>
-                <cylinder radius="0.06" length="0.04"/>
+                <cylinder radius="${wheel_radius}" length="${wheel_length}"/>
             </geometry>
             <material name="blue"/>
@@ -54,11 +75,12 @@
         <collision>
             <geometry>
-                <cylinder radius="0.06" length="0.04"/>
+                <cylinder radius="${wheel_radius}" length="${wheel_length}"/>
             </geometry>
         </collision>
-        <xacro:inertial_cylinder mass="0.1" length="0.04" radius="0.05">
+        <xacro:inertial_cylinder mass="${wheel_mass}" length="${wheel_length}" radius="${wheel_radius}">
             <origin xyz="0 0 0" rpy="0 0 0"/>
         </xacro:inertial_cylinder>
     </link>
+    <!-- Right Wheel -->
     <joint name="right_wheel_joint" type="continuous">
         <parent link="base_link"/>
@@ -70,5 +92,5 @@
         <visual>
             <geometry>
-                <cylinder radius="0.06" length="0.04"/>
+                <cylinder radius="${wheel_radius}" length="${wheel_length}"/>
             </geometry>
             <material name="blue"/>
@@ -76,11 +98,12 @@
         <collision>
             <geometry>
-                <cylinder radius="0.06" length="0.04"/>
+                <cylinder radius="${wheel_radius}" length="${wheel_length}"/>
             </geometry>
         </collision>
-        <xacro:inertial_cylinder mass="0.1" length="0.04" radius="0.05">
+        <xacro:inertial_cylinder mass="${wheel_mass}" length="${wheel_length}" radius="${wheel_radius}">
             <origin xyz="0 0 0" rpy="0 0 0"/>
         </xacro:inertial_cylinder>
     </link>
+    <!-- Caster Wheel -->
     <joint name="caster_wheel_joint" type="fixed">
         <parent link="chassis"/>
@@ -91,5 +114,5 @@
         <visual>
             <geometry>
-                <sphere radius="0.05"/>
+                <sphere radius="${caster_radius}"/>
             </geometry>
             <material name="black"/>
@@ -97,8 +120,8 @@
         <collision>
             <geometry>
-                <sphere radius="0.05"/>
+                <sphere radius="${caster_radius}"/>
             </geometry>
         </collision>
-        <xacro:inertial_sphere mass="0.1" radius="0.05">
+        <xacro:inertial_sphere mass="${caster_mass}" radius="${caster_radius}">
             <origin xyz="0 0 0" rpy="0 0 0"/>
         </xacro:inertial_sphere>
